File: PCB.kicad_pcb (KiCad board)
At the start: 2 copper layers, 150 x 150 mm, 14 parts

Commit message: 2
Connections:
- PicoR1 pad 3: unconnected-(PicoR1-Pin_3-Pad3) -> GND1
- TB6612FNGL1 pad 1: GND -> GND1
Changed lines of the file:
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@@
 	(net 40 "unconnected-(PicoR1-Pin_10-Pad10)")
 	(net 41 "unconnected-(PicoR1-Pin_18-Pad18)")
-	(net 42 "unconnected-(PicoR1-Pin_3-Pad3)")
+	(net 42 "GND1")
 	(net 43 "Net-(PicoR1-Pin_1)")
 	(net 44 "Net-(PicoR1-Pin_7)")
@@
 			(layers "*.Cu" "*.Mask")
 			(remove_unused_layers no)
-			(net 42 "unconnected-(PicoR1-Pin_3-Pad3)")
+			(net 42 "GND1")
 			(pinfunction "Pin_3")
 			(pintype "passive")
@@
 			(layers "*.Cu" "*.Mask")
 			(remove_unused_layers no)
-			(net 2 "GND")
+			(net 42 "GND1")
 			(pinfunction "Pin_1")
 			(pintype "passive")
@@
 	)
 	(segment
+		(start 139.62 112.120293)
+		(end 139.879707 112.120293)
+		(width 1)
+		(layer "F.Cu")
+		(net 36)
+	)
+	(segment
+		(start 139.879707 112.120293)
+		(end 140 112)
+		(width 1)
+		(layer "F.Cu")
+		(net 36)
+	)
+	(segment

Commit message: 3
Parts:
- moved Battery1 71.7 mm to (169.5, 90.8), turned to 180 degrees
- moved Buck_IN-1 66.2 mm to (172.6, 103.5), turned to -90 degrees
- moved Buck_OUT-1 60.7 mm to (172.6, 123.5), turned to -90 degrees
- moved Buck_IN+1 52.8 mm to (162.0, 103.5), turned to -90 degrees
- moved PicoR1 48.1 mm to (139.6, 112.0), turned to 180 degrees
- moved Buck_OUT+1 45.8 mm to (162.0, 123.5), turned to -90 degrees
Connections:
- net GND1 renamed Net-(PicoR1-Pin_3)
- PicoL1 pad 18: unconnected-(PicoL1-Pin_18-Pad18) -> Net-(PicoL1-Pin_18)
- PicoL1 pad 3: GND -> unconnected-(PicoL1-Pin_3-Pad3)
- PicoR1 pad 18: unconnected-(PicoR1-Pin_18-Pad18) -> GND
- TB6612FNGL1 pad 2: Net-(PicoR1-Pin_7) -> Net-(PicoR1-Pin_1)
- TB6612FNGL1 pad 3: Net-(PicoR1-Pin_6) -> Net-(PicoR1-Pin_2)
- TB6612FNGL1 pad 4: Net-(PicoR1-Pin_5) -> Net-(PicoR1-Pin_4)
- TB6612FNGL1 pad 6: Net-(PicoR1-Pin_4) -> Net-(PicoR1-Pin_5)
- TB6612FNGL1 pad 7: Net-(PicoR1-Pin_2) -> Net-(PicoR1-Pin_6)
- TB6612FNGL1 pad 8: Net-(PicoR1-Pin_1) -> Net-(PicoR1-Pin_7)
- TB6612FNGR1 pad 3: GND -> Net-(PicoL1-Pin_18)
- TB6612FNGR1 pad 4: Net-(MotorBR1-Pin_1) -> Net-(MotorBR1-Pin_2)
- TB6612FNGR1 pad 5: Net-(MotorBR1-Pin_2) -> Net-(MotorBR1-Pin_1)
- TB6612FNGR1 pad 6: Net-(MotorBL1-Pin_2) -> Net-(MotorBL1-Pin_1)
- TB6612FNGR1 pad 7: Net-(MotorBL1-Pin_1) -> Net-(MotorBL1-Pin_2)
- TB6612FNGR1 pad 8: GND -> unconnected-(TB6612FNGR1-Pin_8-Pad8)
Routing:
- net Net-(MotorBR1-Pin_2): track 232.9 -> 141.0 mm
- net VCC: track 0.00 -> 77.0 mm
- net GND: track 27.6 -> 99.4 mm
- net /3V3_OUT: track 68.5 -> 19.2 mm
- net Net-(PicoL1-Pin_18): track 0.00 -> 47.8 mm
- net /BuckOut: track 0.00 -> 46.4 mm
- net Net-(PicoR1-Pin_7): track 0.00 -> 40.4 mm
- net Net-(PicoR1-Pin_6): track 0.00 -> 35.8 mm
- net Net-(PicoR1-Pin_5): track 0.00 -> 30.9 mm
- net Net-(PicoR1-Pin_4): track 0.00 -> 24.9 mm
- net Net-(PicoR1-Pin_3): track 0.00 -> 17.5 mm
- net Net-(PicoR1-Pin_2): track 0.00 -> 15.7 mm
- net Net-(MotorBL1-Pin_2): track 143.9 -> 132.2 mm
- net Net-(PicoR1-Pin_1): track 0.00 -> 10.8 mm
- net Net-(MotorBR1-Pin_1): track 138.9 -> 143.3 mm
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
Commit message: v1
1st completed version of PCB
Size is large than needed
Connections:
- PicoL1 pad 13: unconnected-(PicoL1-Pin_13-Pad13) -> GND
- PicoL1 pad 18: Net-(PicoL1-Pin_18) -> GND
- PicoL1 pad 2: unconnected-(PicoL1-Pin_2-Pad2) -> Net-(PicoL1-Pin_2)
- PicoL1 pad 3: unconnected-(PicoL1-Pin_3-Pad3) -> GND
- PicoL1 pad 8: Net-(PicoL1-Pin_8) -> GND
- PicoR1 pad 13: unconnected-(PicoR1-Pin_13-Pad13) -> GND
- PicoR1 pad 3: Net-(PicoR1-Pin_3) -> GND
- PicoR1 pad 8: unconnected-(PicoR1-Pin_8-Pad8) -> GND
- QTR-8RC1 pad 10: Net-(PicoL1-Pin_4) -> Net-(PicoL1-Pin_2)
- QTR-8RC1 pad 6: Net-(PicoL1-Pin_8) -> Net-(PicoL1-Pin_7)
- QTR-8RC1 pad 7: Net-(PicoL1-Pin_7) -> Net-(PicoL1-Pin_6)
- QTR-8RC1 pad 8: Net-(PicoL1-Pin_6) -> Net-(PicoL1-Pin_5)
- QTR-8RC1 pad 9: Net-(PicoL1-Pin_5) -> Net-(PicoL1-Pin_4)
- TB6612FNGL1 pad 1: Net-(PicoR1-Pin_3) -> GND
- TB6612FNGR1 pad 3: Net-(PicoL1-Pin_18) -> GND
- TB6612FNGR1 pad 8: unconnected-(TB6612FNGR1-Pin_8-Pad8) -> GND
Routing:
- net GND: track 99.4 -> 451.5 mm
- net /3V3_OUT: track 19.2 -> 117.4 mm
- net Net-(PicoL1-Pin_8): track 80.8 -> 0.00 mm
- net Net-(PicoL1-Pin_10): track 101.6 -> 48.8 mm
- net Net-(PicoL1-Pin_18): track 47.8 -> 0.00 mm
- net Net-(PicoL1-Pin_9): track 91.2 -> 45.0 mm
- net Net-(PicoL1-Pin_11): track 112.0 -> 74.5 mm
- net Net-(PicoL1-Pin_12): track 122.4 -> 85.0 mm
- net Net-(PicoL1-Pin_7): track 70.4 -> 39.8 mm
- net Net-(PicoL1-Pin_2): track 0.00 -> 24.7 mm
- net /BuckOut: track 46.4 -> 70.2 mm
- net Net-(PicoL1-Pin_6): track 60.0 -> 36.4 mm
- net Net-(PicoR1-Pin_3): track 17.5 -> 0.00 mm
- net Net-(PicoL1-Pin_5): track 49.6 -> 33.1 mm
- net Net-(PicoL1-Pin_4): track 39.1 -> 29.7 mm
