File: PCB.kicad_sch (KiCad schematic)
At the start: 14 parts

Commit message: 2
Connections:
- net GND: no longer TB6612FNGL1.1 (Pin_1)
- net GND1: now reaches PicoR1.18 (Pin_18)
- net GND1: now also TB6612FNGL1.1 (Pin_1)
Changed lines of the file:
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@@
+	)
+	(symbol
+		(lib_id "power:GND")
+		(at 87.63 77.47 0)
+		(unit 1)
+		(exclude_from_sim no)
+		(in_bom yes)
+		(on_board yes)
+		(dnp no)
+		(fields_autoplaced yes)
+		(property "Reference" "#PWR04"
+			(at 87.63 83.82 0)
+			(effects
+				(font
+					(size 1.27 1.27)
+				)
+				(hide yes)
+			)
+		)
+		(property "Value" "GND1"
+			(at 90.17 78.7399 0)
+			(effects
+				(font
+					(size 1.27 1.27)
+				)
+				(justify left)
+			)
+		)
+		(property "Footprint" ""
+			(at 87.63 77.47 0)
+			(effects
+				(font
+					(size 1.27 1.27)
+				)
+				(hide yes)
+			)
+		)
+		(property "Datasheet" ""
+			(at 87.63 77.47 0)
+			(effects
+				(font
+					(size 1.27 1.27)
+				)
+				(hide yes)
+			)
+		)
+		(property "Description" "Power symbol creates a global label with name \"GND\" , ground"
+			(at 87.63 77.47 0)
+			(effects
+				(font
+					(size 1.27 1.27)
+				)
+				(hide yes)
+			)
+		)
+		(pin "1"
+		)
+		(instances
+			(project "PCB"
+				(path "/28f9cef8-479c-4385-8717-8332136a54e7"
+					(reference "#PWR04")
+					(unit 1)
+				)
+			)
+		)
 	)
 	(symbol
@@
 			)
 		)
-		(property "Value" "GND"
-			(at 160.02 99.06 0)
-			(effects
-				(font
-					(size 1.27 1.27)
-				)
-			)
-		)
+		(property "Value" "GND1"
+			(at 162.56 95.2499 0)
+			(effects
+				(font
+					(size 1.27 1.27)
+				)
+				(justify left)
+			)
+		)

Commit message: 3
Connections:
- net GND: now also PicoR1.18 (Pin_18); no longer PicoL1.3 (Pin_3), TB6612FNGR1.3 (Pin_3), TB6612FNGR1.8 (Pin_8)
- net at MotorBL1.1 (Pin_1), MotorFL1.1 (Pin_1): now also TB6612FNGR1.6 (Pin_6); no longer TB6612FNGR1.7 (Pin_7)
- net at MotorBL1.2 (Pin_2), MotorFL1.2 (Pin_2): now also TB6612FNGR1.7 (Pin_7); no longer TB6612FNGR1.6 (Pin_6)
- net at PicoR1.1 (Pin_1): now also TB6612FNGL1.2 (Pin_2); no longer TB6612FNGL1.8 (Pin_8)
- net at PicoR1.2 (Pin_2): now also TB6612FNGL1.3 (Pin_3); no longer TB6612FNGL1.7 (Pin_7)
- net at PicoR1.3 (Pin_3): now also TB6612FNGL1.1 (Pin_1)
- net at PicoR1.4 (Pin_4): now also TB6612FNGL1.4 (Pin_4); no longer TB6612FNGL1.6 (Pin_6)
- net at PicoR1.5 (Pin_5): now also TB6612FNGL1.6 (Pin_6); no longer TB6612FNGL1.4 (Pin_4)
- net at PicoR1.6 (Pin_6): now also TB6612FNGL1.7 (Pin_7); no longer TB6612FNGL1.3 (Pin_3)
- net at PicoR1.7 (Pin_7): now also TB6612FNGL1.8 (Pin_8); no longer TB6612FNGL1.2 (Pin_2)
- net at MotorBR1.1 (Pin_1), MotorFR1.1 (Pin_1): now also TB6612FNGR1.5 (Pin_5); no longer TB6612FNGR1.4 (Pin_4)
- net at MotorBR1.2 (Pin_2), MotorFR1.2 (Pin_2): now also TB6612FNGR1.4 (Pin_4); no longer TB6612FNGR1.5 (Pin_5)
- net at PicoL1.18 (Pin_18): now also TB6612FNGR1.3 (Pin_3)
- removed net GND1: PicoR1.18 (Pin_18), TB6612FNGL1.1 (Pin_1)
Other:
- moved on the sheet: TB6612FNGL1

Commit message: v1
1st completed version of PCB
Size is large than needed
Connections:
- net GND: now also PicoL1.13 (Pin_13), PicoL1.18 (Pin_18), PicoL1.3 (Pin_3), PicoL1.8 (Pin_8), PicoR1.13 (Pin_13), PicoR1.3 (Pin_3), PicoR1.8 (Pin_8), TB6612FNGL1.1 (Pin_1), TB6612FNGR1.3 (Pin_3), TB6612FNGR1.8 (Pin_8)
- net at QTR-8RC1.10 (Pin_10): now also PicoL1.2 (Pin_2); no longer PicoL1.4 (Pin_4)
- net at QTR-8RC1.6 (Pin_6): now also PicoL1.7 (Pin_7); no longer PicoL1.8 (Pin_8)
- net at QTR-8RC1.7 (Pin_7): now also PicoL1.6 (Pin_6); no longer PicoL1.7 (Pin_7)
- net at QTR-8RC1.8 (Pin_8): now also PicoL1.5 (Pin_5); no longer PicoL1.6 (Pin_6)
- net at QTR-8RC1.9 (Pin_9): now also PicoL1.4 (Pin_4); no longer PicoL1.5 (Pin_5)
Other:
- moved on the sheet: QTR-8RC1
