File: PCB/PCB.kicad_pcb (KiCad board)
At the start: 2 copper layers, 75 x 75 mm, 14 parts

Commit message: 100x100
Parts:
- moved TB6612FNGR1 131.2 mm to (135.0, 80.1), turned to -90 degrees
- moved MotorBR1 130.2 mm to (159.8, 8.80)
- moved TB6612FNGL1 113.1 mm to (135.0, 64.0), turned to -90 degrees
- moved MotorFR1 97.6 mm to (159.8, 56.6)
- moved MotorBL1 94.2 mm to (81.8, 7.75), turned to 0 degrees
- moved QTR-8RC1 89.3 mm to (139.1, -10.0)
- moved Buck_IN+1 86.7 mm to (144.0, 25.0)
- moved Buck_OUT+1 86.7 mm to (144.0, 45.0)
- moved Buck_IN-1 86.7 mm to (154.5, 25.0)
- moved Buck_OUT-1 86.7 mm to (154.5, 45.0)
- moved PicoL1 86.3 mm to (115.0, 6.69)
- moved PicoR1 86.3 mm to (132.6, 54.8)
- moved Battery1 86.0 mm to (150.5, 13.0)
- moved MotorFL1 54.4 mm to (81.8, 55.5), turned to 0 degrees
Routing:
- net VCC: track 125.2 -> 74.1 mm, vias 2 -> 1
- net Net-(MotorBL1-Pin_1): track 48.8 -> 98.5 mm
- net Net-(MotorBL1-Pin_2): track 49.4 -> 90.9 mm, vias 0 -> 1
- net Net-(PicoR1-Pin_7): track 58.4 -> 30.8 mm, vias 1 -> 0
- net Net-(PicoR1-Pin_6): track 54.2 -> 27.2 mm
- net Net-(PicoR1-Pin_5): track 47.6 -> 23.6 mm, vias 1 -> 0
- net Net-(MotorBR1-Pin_2): track 71.6 -> 95.0 mm
- net Net-(PicoR1-Pin_1): track 32.1 -> 9.24 mm
- net Net-(PicoR1-Pin_2): track 33.9 -> 13.0 mm
- net Net-(PicoR1-Pin_4): track 36.9 -> 19.0 mm, vias 0 -> 1
- net Net-(MotorBR1-Pin_1): track 77.8 -> 92.5 mm, vias 1 -> 0
- net /3V3_OUT: track 111.5 -> 99.1 mm, vias 2 -> 1
- net Net-(PicoL1-Pin_7): track 26.9 -> 36.6 mm
- net Net-(PicoL1-Pin_6): track 23.3 -> 33.0 mm
- net Net-(PicoL1-Pin_5): track 19.7 -> 29.5 mm
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Other:
- board size 75 x 75 mm -> 100 x 100 mm

Commit message: 100x100
Parts:
- moved Buck_IN+1 75.0 mm to (70.6, 40.6)
- moved Buck_OUT+1 75.0 mm to (70.6, 60.6)
- moved MotorBL1 75.0 mm to (8.35, 23.4)
- moved MotorBR1 75.0 mm to (86.4, 24.4)
- moved MotorFR1 75.0 mm to (86.4, 72.2)
- moved TB6612FNGR1 75.0 mm to (61.6, 95.7)
- moved Battery1 75.0 mm to (77.1, 28.6)
- moved Buck_IN-1 75.0 mm to (81.1, 40.6)
- moved Buck_OUT-1 75.0 mm to (81.1, 60.6)
- moved MotorFL1 75.0 mm to (8.35, 71.1)
- moved PicoL1 75.0 mm to (41.6, 22.3)
- moved PicoR1 75.0 mm to (59.2, 70.4)
- moved QTR-8RC1 75.0 mm to (65.7, 5.60)
- moved TB6612FNGL1 75.0 mm to (61.6, 79.6)
Routing:
- net /3V3_OUT: track 99.1 -> 98.2 mm
- net VCC: track 74.1 -> 73.2 mm
- net GND18: track 37.2 -> 36.7 mm
- net Net-(PicoL1-Pin_11): track 50.0 -> 49.4 mm
- net Net-(PicoL1-Pin_10): track 46.4 -> 45.8 mm
- net Net-(PicoL1-Pin_9): track 42.8 -> 42.2 mm
- net Net-(PicoL1-Pin_12): track 53.5 -> 53.0 mm
- net Net-(PicoL1-Pin_5): track 29.5 -> 28.9 mm

Commit message: screw holes
Parts:
- added H1: MountingHole, MountingHole:MountingHole_3.2mm_M3, F.Cu at (9.00, 9.00)
- added H2: MountingHole, MountingHole:MountingHole_3.2mm_M3, F.Cu at (91.0, 9.00)
- added H3: MountingHole, MountingHole:MountingHole_3.2mm_M3, F.Cu at (9.00, 91.0)
- added H4: MountingHole, MountingHole:MountingHole_3.2mm_M3, F.Cu at (91.0, 91.0)
