File: PCB/PCB.kicad_sch (KiCad schematic)
At the start: 18 parts

Commit message: 100x100 pdf
Connections:
- net 3V3_OUT: no longer TB6612FNGL1.5 (Pin_5)
Changed lines of the file:
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@@
-		)
-	)
-	(label "3V3_OUT"
-		(at 95.25 111.76 180)
-		(effects
-			(font
-				(size 1.27 1.27)
-			)
-			(justify right bottom)
 		)
 	)

Commit message: 75x75
Parts:
- removed H1, H2, H3, H4: MountingHole, MountingHole:MountingHole_3.2mm_M3, symbol Mechanical:MountingHole
Connections:
- net 3V3_OUT: now also TB6612FNGL1.5 (Pin_5)
Other:
- moved on the sheet: Battery1, Buck_IN+1, Buck_IN-1, Buck_OUT+1, Buck_OUT-1
